File: Hardware/MOTOR_DRIVE.kicad_sch (KiCad schematic)
At the start: 14 parts, among them J6 Conn_01x03, J7 Conn_01x06, J8 Conn_01x06, U3 DRV8833PWP

Commit message: Schematic update
Other:
- title: (none) -> MCU_AND_SENSORS
Changed lines of the file:
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@@
 	(generator_version "10.0")
 	(paper "A4")
+	(title_block
+		(title "MCU_AND_SENSORS")
+		(date "2026-09-20")
+	)
 	(text "Servo Connector"
 		(exclude_from_sim no)
