File: Hardware/POWER_MANAGEMENT.kicad_sch (KiCad schematic)
At the start: 54 parts, among them J4 USB_C_Receptacle_USB2.0_16P, J5 Conn_01x02_Pin, Q1 2N7002, Q2 Q_PMOS, Q5 Q_PNP_CurrentMirror, U4 AP2112K-3.3, U5 bq27220, U9 BQ25896RTWR

Commit message: Schematic update
Other:
- title: (none) -> MCU_AND_SENSORS
Changed lines of the file:
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@@
 	(generator_version "10.0")
 	(paper "A4")
+	(title_block
+		(title "MCU_AND_SENSORS")
+		(date "2026-09-20")
+	)
 	(text "Battery charger "
 		(exclude_from_sim no)
