File: Hardware/SENSORS.kicad_sch (KiCad schematic)
At the start: 17 parts, among them J1 Conn_01x04_Pin, J10 Conn_01x06, J11 Conn_01x06, J12 Conn_01x06, J3 C573320, U2 MPU-6050

Commit message: Schematic update
Other:
- title: (none) -> MCU_AND_SENSORS
Changed lines of the file:
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@@
 	(generator_version "10.0")
 	(paper "A4")
+	(title_block
+		(title "MCU_AND_SENSORS")
+		(date "2026-09-20")
+	)
 	(text ""
 		(exclude_from_sim no)
