File: Hardware/robot_canettes.kicad_sch (KiCad schematic)
At the start: 0 parts

Commit message: Schematic update
Other:
- title: (none) -> MCU_AND_SENSORS
Changed lines of the file:
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@@
 	(generator_version "10.0")
 	(paper "A4")
+	(title_block
+		(title "MCU_AND_SENSORS")
+		(date "2026-09-20")
+	)
 	(wire
 		(pts
